Commit message: pid with drive

File: src/my_bot/description/robot.urdf.xacro (robot description, xacro)
@@ -2,5 +2,4 @@
 <robot name="my_bot" xmlns:xacro="http://ros.org/wiki/xacro">
     <xacro:include filename="inertial_macros.xacro"/>
-    <xacro:include filename="gazebo_control.xacro"/>
     <xacro:include filename="robot_core.xacro"/>
     <xacro:include filename="lidar.xacro"/>

File: src/my_bot/description/robot_core.xacro (robot description, xacro)
@@ -27,5 +27,5 @@
             <origin xyz="0.15 0.0 0.075"/>
             <geometry>
-                <box size="0.3 0.3 0.15"/>
+                <box size="0.3 0.23 0.08"/>
             </geometry>
             <material name="white"/>
@@ -44,5 +44,5 @@
         <material>Gazebo/White</material>
     </gazebo>
-    <!-- Left Wheel Link -->
+    <!-- Left Wheel Joint -->
     <joint name = "left_wheel_joint" type = "continuous">
         <parent link = "base_link"/>
@@ -51,8 +51,9 @@
         <axis xyz = "0 0 1"/>
     </joint>
+    <!-- Left Wheel Link-->
     <link name = "left_wheel">
         <visual>
             <geometry>
-                <cylinder radius="0.05" length="0.04"/>
+                <cylinder radius="0.03" length="0.07"/>
             </geometry>
             <material name='blue' />
@@ -60,5 +61,5 @@
         <collision>
             <geometry>
-                <cylinder radius="0.05" length="0.04"/>
+                <cylinder radius="0.03" length="0.07"/>
             </geometry>
         </collision>
@@ -70,5 +71,5 @@
         <material>Gazebo/Blue</material>
     </gazebo>
-    <!-- Right Wheel Link -->
+    <!-- Right Wheel Joint -->
     <joint name = "right_wheel_joint" type = "continuous">
         <parent link = "base_link"/>
@@ -77,8 +78,9 @@
         <axis xyz = "0 0 -1"/>
     </joint>
+    <!-- Right Wheel Link -->
     <link name = "right_wheel">
         <visual>
             <geometry>
-                <cylinder radius="0.05" length="0.04"/>
+                <cylinder radius="0.03" length="0.07"/>
             </geometry>
             <material name='blue' />
@@ -86,5 +88,5 @@
         <collision>
             <geometry>
-                <cylinder radius="0.05" length="0.04"/>
+                <cylinder radius="0.03" length="0.07"/>
             </geometry>
             <material name='blue' />
