Commit message: slam implementation

File: src/my_bot/description/lidar.xacro (robot description, xacro)
@@ -24,5 +24,5 @@
     <gazebo reference="lidar_link">
         <material>Gazebo/Red</material>
-        <sensor type="ray" name="lidar_sensor">
+        <!-- <sensor type="ray" name="lidar_sensor">
             <pose>0 0 0 0 0 0</pose>
             <visualize>true</visualize>
@@ -51,5 +51,5 @@
                 </ros>
             </plugin>
-        </sensor>
+        </sensor> -->
     </gazebo>
 </robot>

File: src/my_bot/description/robot_core.xacro (robot description, xacro)
@@ -16,4 +16,11 @@
     <!-- Base Link -->
     <link name = "base_link">
+    </link>
+    <joint name = "base_footprint_joint" type="fixed">
+        <parent link="base_link"/>
+        <child link="base_footprint"/>
+        <origin xyz="0 0 0" rpy="0 0 0"/>
+    </joint>
+    <link name = "base_footprint">
     </link>
     <!-- Chassis Link -->

Commit message: changes to slam

File: src/my_bot/description/lidar.xacro (robot description, xacro)
@@ -2,7 +2,7 @@
 <robot xmlns:xacro="http://www.ros.org/wiki/xacro">
     <joint name="lidar_joint" type="fixed">
-        <parent link="chassis"/>
+        <parent link="base_link"/>
         <child link="lidar_link"/>
-        <origin xyz="0.15 0 0.15" rpy="0 0 0"/>
+        <origin xyz="0.15 0 0.15" rpy="0 0 -1.570795"/>
     </joint>
     <link name="lidar_link">
